Commit message: update from upstream

File: iiwa_description/urdf/iiwa.transmission.xacro (robot description, xacro)
@@ -3,4 +3,5 @@
   <xacro:macro name="iiwa_transmission" params="hardware_interface">
     <transmission name="${robot_name}_tran_1">
+      <robotNamespace>/${robot_name}</robotNamespace>
       <type>transmission_interface/SimpleTransmission</type>
       <joint name="${robot_name}_joint_1">
@@ -8,8 +9,10 @@
       </joint>
       <actuator name="${robot_name}_motor_1">
+        <hardwareInterface>hardware_interface/${hardware_interface}</hardwareInterface>
         <mechanicalReduction>1</mechanicalReduction>
       </actuator>
     </transmission>
     <transmission name="${robot_name}_tran_2">
+      <robotNamespace>/${robot_name}</robotNamespace>
       <type>transmission_interface/SimpleTransmission</type>
       <joint name="${robot_name}_joint_2">
@@ -17,8 +20,10 @@
       </joint>
       <actuator name="${robot_name}_motor_2">
+        <hardwareInterface>hardware_interface/${hardware_interface}</hardwareInterface>
         <mechanicalReduction>1</mechanicalReduction>
       </actuator>
     </transmission>
     <transmission name="${robot_name}_tran_3">
+      <robotNamespace>/${robot_name}</robotNamespace>
       <type>transmission_interface/SimpleTransmission</type>
       <joint name="${robot_name}_joint_3">
@@ -26,8 +31,10 @@
       </joint>
       <actuator name="${robot_name}_motor_3">
+        <hardwareInterface>hardware_interface/${hardware_interface}</hardwareInterface>
         <mechanicalReduction>1</mechanicalReduction>
       </actuator>
     </transmission>
     <transmission name="${robot_name}_tran_4">
+      <robotNamespace>/${robot_name}</robotNamespace>
       <type>transmission_interface/SimpleTransmission</type>
       <joint name="${robot_name}_joint_4">
@@ -35,8 +42,10 @@
       </joint>
       <actuator name="${robot_name}_motor_4">
+        <hardwareInterface>hardware_interface/${hardware_interface}</hardwareInterface>
         <mechanicalReduction>1</mechanicalReduction>
       </actuator>
     </transmission>
     <transmission name="${robot_name}_tran_5">
+      <robotNamespace>/${robot_name}</robotNamespace>
       <type>transmission_interface/SimpleTransmission</type>
       <joint name="${robot_name}_joint_5">
@@ -44,8 +53,10 @@
       </joint>
       <actuator name="${robot_name}_motor_5">
+        <hardwareInterface>hardware_interface/${hardware_interface}</hardwareInterface>
         <mechanicalReduction>1</mechanicalReduction>
       </actuator>
     </transmission>
     <transmission name="${robot_name}_tran_6">
+      <robotNamespace>/${robot_name}</robotNamespace>
       <type>transmission_interface/SimpleTransmission</type>
       <joint name="${robot_name}_joint_6">
@@ -53,8 +64,10 @@
       </joint>
       <actuator name="${robot_name}_motor_6">
+        <hardwareInterface>hardware_interface/${hardware_interface}</hardwareInterface>
         <mechanicalReduction>1</mechanicalReduction>
       </actuator>
     </transmission>
     <transmission name="${robot_name}_tran_7">
+      <robotNamespace>/${robot_name}</robotNamespace>
       <type>transmission_interface/SimpleTransmission</type>
       <joint name="${robot_name}_joint_7">
@@ -62,4 +75,5 @@
       </joint>
       <actuator name="${robot_name}_motor_7">
+        <hardwareInterface>hardware_interface/${hardware_interface}</hardwareInterface>
         <mechanicalReduction>1</mechanicalReduction>
       </actuator>

File: iiwa_description/urdf/iiwa14.xacro (robot description, xacro)
@@ -38,11 +38,12 @@
           <mesh filename="package://iiwa_description/meshes/iiwa14/collision/link_0.stl"/>
         </geometry>
-      </collision>
-      <!-- <self_collision_checking>
+        <material name="Grey"/>
+      </collision>
+      <self_collision_checking>
         <origin xyz="0 0 0" rpy="0 0 0"/>
         <geometry>
           <capsule radius="0.15" length="0.25"/>
         </geometry>
-      </self_collision_checking> -->
+      </self_collision_checking>
     </link>
     <!-- joint between link_0 and link_1 -->
@@ -78,4 +79,5 @@
           <mesh filename="package://iiwa_description/meshes/iiwa14/collision/link_1.stl"/>
         </geometry>
+        <material name="Orange"/>
       </collision>
     </link>
@@ -112,4 +114,5 @@
           <mesh filename="package://iiwa_description/meshes/iiwa14/collision/link_2.stl"/>
         </geometry>
+        <material name="Orange"/>
       </collision>
     </link>
@@ -146,4 +149,5 @@
           <mesh filename="package://iiwa_description/meshes/iiwa14/collision/link_3.stl"/>
         </geometry>
+        <material name="Orange"/>
       </collision>
     </link>
@@ -180,4 +184,5 @@
           <mesh filename="package://iiwa_description/meshes/iiwa14/collision/link_4.stl"/>
         </geometry>
+        <material name="Orange"/>
       </collision>
     </link>
@@ -214,4 +219,5 @@
           <mesh filename="package://iiwa_description/meshes/iiwa14/collision/link_5.stl"/>
         </geometry>
+        <material name="Orange"/>
       </collision>
     </link>
@@ -248,4 +254,5 @@
           <mesh filename="package://iiwa_description/meshes/iiwa14/collision/link_6.stl"/>
         </geometry>
+        <material name="Orange"/>
       </collision>
     </link>
@@ -282,4 +289,5 @@
           <mesh filename="package://iiwa_description/meshes/iiwa14/collision/link_7.stl"/>
         </geometry>
+        <material name="Grey"/>
       </collision>
     </link>

File: iiwa_description/urdf/iiwa7.xacro (robot description, xacro)
@@ -38,11 +38,12 @@
           <mesh filename="package://iiwa_description/meshes/iiwa7/collision/link_0.stl"/>
         </geometry>
-      </collision>
-      <!-- <self_collision_checking>
+        <material name="Grey"/>
+      </collision>
+      <self_collision_checking>
         <origin xyz="0 0 0" rpy="0 0 0"/>
         <geometry>
           <capsule radius="0.15" length="0.25"/>
         </geometry>
-      </self_collision_checking> -->
+      </self_collision_checking>
     </link>
     <!-- joint between link_0 and link_1 -->
@@ -78,4 +79,5 @@
           <mesh filename="package://iiwa_description/meshes/iiwa7/collision/link_1.stl"/>
         </geometry>
+        <material name="Orange"/>
       </collision>
     </link>
@@ -111,4 +113,5 @@
           <mesh filename="package://iiwa_description/meshes/iiwa7/collision/link_2.stl"/>
         </geometry>
+        <material name="Orange"/>
       </collision>
     </link>
@@ -144,4 +147,5 @@
           <mesh filename="package://iiwa_description/meshes/iiwa7/collision/link_3.stl"/>
         </geometry>
+        <material name="Orange"/>
       </collision>
     </link>
@@ -177,4 +181,5 @@
           <mesh filename="package://iiwa_description/meshes/iiwa7/collision/link_4.stl"/>
         </geometry>
+        <material name="Orange"/>
       </collision>
     </link>
@@ -210,4 +215,5 @@
           <mesh filename="package://iiwa_description/meshes/iiwa7/collision/link_5.stl"/>
         </geometry>
+        <material name="Orange"/>
       </collision>
     </link>
@@ -243,4 +249,5 @@
           <mesh filename="package://iiwa_description/meshes/iiwa7/collision/link_6.stl"/>
         </geometry>
+        <material name="Orange"/>
       </collision>
     </link>
@@ -276,4 +283,5 @@
           <mesh filename="package://iiwa_description/meshes/iiwa7/collision/link_7.stl"/>
         </geometry>
+        <material name="Grey"/>
       </collision>
     </link>
